File: Chimaera_DSP-F3_Unit.sch (KiCad schematic (older format))
At the start: 44 parts, among them J1 USB_MINI, P1 power in, P11 CONN_6, P2 from sensor units, P3 from sensor units, P5 to sensor units, SW1 DPDT, U1 LM1117, U2 MCP1703, U3 MCP1754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

Commit message: bug-fix in DSP with wrongly wired I2C2
Parts:
- removed U4: F303Cx, MODULE, symbol STM32F303XX
- added P12: CONN_2, ~, symbol CONN_2
- added U4: STM32F303CX, MODULE, symbol STM32F303CX
Connections:
- wire segments 82 -> 72
Other:
- moved on the sheet: P11

Commit message: EDA: all resistors now in 0603 format
Parts:
- R1, R2, R4: Digi-Key P1.05KCCT-ND -> P1.0KGCT-ND
- R3, R5: Digi-Key P10.2KCCT-ND -> P10KGCT-ND
- R6, R7: Digi-Key P4.75KCCT-ND -> P4.75KHCT-ND
- R8: Digi-Key P1.50KCCT-ND -> P1.50KHCT-ND
Changed lines of the file:
@@
 Sheet 1 2
 Title "Chimaera DSP Unit"
-Date "29 nov 2013"
+Date "5 dec 2013"
 Rev "4"
 Comp "by Open Music Kontrollers (www.open-music-kontrollers.ch)"
@@
 F 2 "" H 12600 2350 60  0000 C CNN
 F 3 "" H 12600 2350 60  0000 C CNN
-F 4 "P10.2KCCT-ND" V 12600 2350 60  0001 C CNN "Digi-Key"
+F 4 "P10KGCT-ND" V 12600 2350 60  0001 C CNN "Digi-Key"
 	1    12600 2350
 	-1   0    0    1
@@
 F 2 "" H 7500 7150 60  0000 C CNN
 F 3 "" H 7500 7150 60  0000 C CNN
-F 4 "P4.75KCCT-ND" V 7500 7150 60  0001 C CNN "Digi-Key"
+F 4 "P4.75KHCT-ND" V 7500 7150 60  0001 C CNN "Digi-Key"
 	1    7500 7150
 	0    -1   -1   0
@@
 F 2 "" H 7500 7350 60  0000 C CNN
 F 3 "" H 7500 7350 60  0000 C CNN
-F 4 "P4.75KCCT-ND" V 7500 7350 60  0001 C CNN "Digi-Key"
+F 4 "P4.75KHCT-ND" V 7500 7350 60  0001 C CNN "Digi-Key"
 	1    7500 7350
 	0    -1   -1   0
@@
 F 2 "" H 11600 2350 60  0000 C CNN
 F 3 "" H 11600 2350 60  0000 C CNN
-F 4 "P1.05KCCT-ND" V 11600 2350 60  0001 C CNN "Digi-Key"
+F 4 "P1.0KGCT-ND" V 11600 2350 60  0001 C CNN "Digi-Key"
 	1    11600 2350
 	1    0    0    -1
@@
 F 2 "" H 12600 1450 60  0000 C CNN
 F 3 "" H 12600 1450 60  0000 C CNN
-F 4 "P10.2KCCT-ND" V 12600 1450 60  0001 C CNN "Digi-Key"
+F 4 "P10KGCT-ND" V 12600 1450 60  0001 C CNN "Digi-Key"
 	1    12600 1450
 	-1   0    0    1
@@
 F 2 "" H 11600 1450 60  0000 C CNN
 F 3 "" H 11600 1450 60  0000 C CNN
-F 4 "P1.05KCCT-ND" V 11600 1450 60  0001 C CNN "Digi-Key"
+F 4 "P1.0KGCT-ND" V 11600 1450 60  0001 C CNN "Digi-Key"
 	1    11600 1450
 	-1   0    0    1
@@
 F 2 "" H 10500 1950 60  0000 C CNN
 F 3 "" H 10500 1950 60  0000 C CNN
-F 4 "P1.05KCCT-ND" V 10500 1950 60  0001 C CNN "Digi-Key"
+F 4 "P1.0KGCT-ND" V 10500 1950 60  0001 C CNN "Digi-Key"
 	1    10500 1950
 	0    -1   -1   0
@@
 F 2 "" H 9050 4350 60  0000 C CNN
 F 3 "" H 9050 4350 60  0000 C CNN
-F 4 "P1.50KCCT-ND" V 9050 4350 60  0001 C CNN "Digi-Key"
+F 4 "P1.50KHCT-ND" V 9050 4350 60  0001 C CNN "Digi-Key"
 	1    9050 4350
 	1    0    0    -1

Commit message: EDA: add missing Digi-Key part numbers
Parts:
- U4: Digi-Key (none) -> 497-13318-ND
Changed lines of the file:
@@
 Sheet 1 2
 Title "Chimaera DSP Unit"
-Date "5 dec 2013"
+Date "2 jan 2014"
 Rev "4"
 Comp "by Open Music Kontrollers (www.open-music-kontrollers.ch)"
@@
 F 2 "MODULE" H 13450 5500 50  0001 C CNN
 F 3 "DOCUMENTATION" H 13450 5500 50  0001 C CNN
+F 4 "497-13318-ND" H 13450 5500 60  0001 C CNN "Digi-Key"
 	1    13450 5500
 	1    0    0    -1
