File: chimaera_dsp_unit.kicad_pcb (KiCad board)
At the start: 2 copper layers, 80 x 44 mm, 89 parts, among them J1 USB_MINI, J51 RJ45-TRANSFO, P1 power in, P11 CONN_6, P12 CONN_2, P2 from sensor units, P3 from sensor units, P5 to sensor units, SW1 DPDT, U1 LM1117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

Commit message: 3.3V version of Revision 4
Parts:
- removed C20: 10uF, SM0805
- removed U3: MCP1754, SOT23
- U6: value 74HCT163 -> 74HC163
Connections:
- C22 pad 2: +5V -> +3.3V
- U6 pad 16: +5V -> +3.3V
Routing:
- net N-0000042: track 133.2 -> 121.9 mm
- net +5V: track 7.54 -> 0.00 mm
- net GND: track 194.8 -> 192.7 mm, vias 65 -> 63
Other:
- board text added: "1"
- board text added: "2"
- board text added: "3"
- board text added: "4"
- board text added: "5"
- board text added: "6"
- board text added: "7"
- board text added: "8"
- board text added: "9"
- board text added: "A"
- board text added: "CHIMAERA DSP Unit Rev4-3v3 with... ST's F303Cx & WIZnet's W5500 -------------------- (c) 2014 Hanspeter Portner Licensed under CERN OHL v.1.2 by Open Music Kontrollers www.open-music-kontrollers.ch"
- board text removed: "CHIMAERA DSP Unit Rev4 with... ST's F303Cx & WIZnet's W5500 -------------------- (c) 2013 Hanspeter Portner Licensed under CERN OHL v.1.2 by Open Music Kontrollers www.open-music-kontrollers.ch"

Commit message: update 3v3 version
Parts:
- added G3: OMK_LOGO, OMK_LOGO, F.Cu at (25.2, 27.8)
- renumbered G*** to G1, G*** to G2
