File: chimaera_dsp_unit.sch (KiCad schematic (older format))
At the start: 45 parts, among them J1 USB_MINI, P1 power in, P11 CONN_6, P12 CONN_2, P2 from sensor units, P3 from sensor units, P5 to sensor units, SW1 DPDT, U1 LM1117, U2 MCP1703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

Commit message: 3.3V version of Revision 4
Parts:
- removed C20: 10uF, symbol C
- removed U3: MCP1754, symbol LM1117
- U6: value 74HCT163 -> 74HC163
Connections:
- net labels removed: +5V
- wire segments 72 -> 69

Commit message: update 3v3 version
Parts:
- U6: Digi-Key 296-33134-5-ND -> 296-33034-5-ND
Changed lines of the file:
@@
 Sheet 1 2
 Title "Chimaera DSP Unit"
-Date "20 apr 2014"
+Date "5 may 2014"
 Rev "4-3v3"
 Comp "by Open Music Kontrollers (www.open-music-kontrollers.ch)"
@@
 F 2 "~" H 10350 7300 60  0000 C CNN
 F 3 "~" H 10350 7300 60  0000 C CNN
-F 4 "296-33134-5-ND" H 10350 7300 60  0001 C CNN "Digi-Key"
+F 4 "296-33034-5-ND" H 10350 7300 60  0001 C CNN "Digi-Key"
 	1    10350 7300
 	1    0    0    -1
